File: pcb/design/01_module_references_v2/03_sulfur_monitoring_references.kicad_sch (KiCad schematic)
At the start: 11 parts, among them U1 Micro_SDCARD_v1, U2 Anemometer, U3 Wind_Direction, U4 Micro_SDCARD_v2, U5 Heltec_WSL_V3

Commit message: renamed symbol to libraries
Parts:
- I1: symbol myCustom_STAS_RG:INA219 -> Library:INA219
- I2: symbol myCustom_STAS_RG:TB600B -> Library:TB600B
- I3: symbol myCustom_STAS_RG:TB600C -> Library:TB600C
- I4: symbol myCustom_STAS_RG:SSD1306​ -> Library:SSD1306​
- I5: symbol myCustom_STAS_RG:GPS -> Library:GPS
- I6: symbol myCustom_STAS_RG:RTC_DS3231​ -> Library:RTC_DS3231​
- U1: symbol myCustom_STAS_RG:SPI SD Card -> Library:SPI SD Card
- U2: symbol myCustom_STAS_RG:Anemometer -> Library:Anemometer
- U3: symbol myCustom_STAS_RG:Wind Direction -> Library:Wind Direction
- U4: symbol myCustom_STAS_RG:SPI SD Card_v2 -> Library:SPI SD Card_v2
- U5: symbol myCustom_STAS_RG:WSL_V3 -> Library:WSL_V3
Changed lines of the file:
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@@
 	)
 	(symbol
-		(lib_id "myCustom_STAS_RG:WSL_V3")
+		(lib_id "Library:WSL_V3")
 		(at 163.83 43.18 0)
 		(unit 1)
@@
 	)
 	(symbol
-		(lib_id "myCustom_STAS_RG:Anemometer")
+		(lib_id "Library:Anemometer")
 		(at 73.66 41.91 0)
 		(unit 1)
@@
 	)
 	(symbol
-		(lib_id "myCustom_STAS_RG:SSD1306​")
+		(lib_id "Library:SSD1306​")
 		(at 110.49 68.58 0)
 		(unit 1)
@@
 	)
 	(symbol
-		(lib_id "myCustom_STAS_RG:INA219")
+		(lib_id "Library:INA219")
 		(at 96.52 69.85 0)
 		(unit 1)
@@
 	)
 	(symbol
-		(lib_id "myCustom_STAS_RG:TB600B")
+		(lib_id "Library:TB600B")
 		(at 29.21 41.91 0)
 		(unit 1)
@@
 	)
 	(symbol
-		(lib_id "myCustom_STAS_RG:TB600C")
+		(lib_id "Library:TB600C")
 		(at 44.45 41.91 0)
 		(unit 1)
@@
 	)
 	(symbol
-		(lib_id "myCustom_STAS_RG:GPS")
+		(lib_id "Library:GPS")
 		(at 58.42 41.91 0)
 		(unit 1)
@@
 	)
 	(symbol
-		(lib_id "myCustom_STAS_RG:SPI SD Card")
+		(lib_id "Library:SPI SD Card")
 		(at 60.96 73.66 0)
 		(unit 1)
@@
 	)
 	(symbol
-		(lib_id "myCustom_STAS_RG:RTC_DS3231​")
+		(lib_id "Library:RTC_DS3231​")
 		(at 36.83 74.93 0)
 		(unit 1)
@@
 	)
 	(symbol
-		(lib_id "myCustom_STAS_RG:Wind Direction")
+		(lib_id "Library:Wind Direction")
 		(at 88.9 41.91 0)
 		(unit 1)
@@
 	)
 	(symbol
-		(lib_id "myCustom_STAS_RG:SPI SD Card_v2")
+		(lib_id "Library:SPI SD Card_v2")
 		(at 80.01 73.66 0)
 		(unit 1)
