File: pcb/design/04_sulfurmonitoring_design_v1/template_spectra_v1.kicad_pcb (KiCad board)
At the start: 2 copper layers, 52.1 x 69.8 mm, 3 parts, among them U1 Heltec_WSL_V3

Commit message: design
Parts:
- removed D1, D2: LED, LED_THT:LED_D5.0mm
- added I1: TB600B SO2, Custom Board:TB600B_SO2, F.Cu at (118.1, 165.1)
- added I2: TB600C_H2S, Custom Board:TB600C_H2S, F.Cu at (118.2, 154.9)
- added I3: uBlox_NEO-6M, Custom Board:uBlox_NEO-6M, F.Cu at (118.2, 124.5)
- added I4: SSD1306​, Custom Board:SSD1306_onBoard, F.Cu at (85.1, 110.5)
- added I5: INA219, Custom Board:INA219, F.Cu at (113.0, 108.0)
- added I6: DS3231​, Custom Board:DS3231, F.Cu at (55.9, 115.8)
- added U2: Anemometer, Custom Board:STASRG_Anemometer, F.Cu at (118.2, 144.8)
- added U3: Micro_SDCARD_v2, Custom Board:Micro_SDCARD_v2, F.Cu at (85.3, 134.3)
- added U4: Wind_Direction, Custom Board:STASRG_Wind_Dir, F.Cu at (118.2, 134.6)
- moved U1 87.5 mm to (73.7, 157.5), turned to -90 degrees
Connections:
- U1 pad 18: Net-(D1-A) -> unconnected-(U1-1-Pad18)
- U1 pad 2: GND -> unconnected-(U1-GND-Pad2)
- U1 pad 23: GND -> unconnected-(U1-GND-Pad23)
- U1 pad 40: Net-(D2-A) -> unconnected-(U1-4-Pad40)
Routing:
- net GND: track 77.7 -> 0.00 mm, vias 1 -> 0
- net Net-(D2-A): track 48.6 -> 0.00 mm
- net Net-(D1-A): track 47.5 -> 0.00 mm
Other:
- board size 52.1 x 69.8 mm -> 90 x 150 mm

Commit message: added revision
Parts:
- added D1: LED, LED_THT:LED_D5.0mm, F.Cu at (198.1, 114.3)
- added D2: LED, LED_THT:LED_D5.0mm, F.Cu at (193.0, 132.1)
- added U5: W5500_Module, Custom Board:W5500_Module, F.Cu at (178.7, 107.8)
- added U6: BUCK_MP1584_3V3, Custom Board:BUCK_MP1584_3V3_Module, F.Cu at (177.3, 131.6)
- I3: footprint Custom Board:uBlox_NEO-6M -> Custom Board:uBlox_NEO-6M_JST
- moved I3 0.12 mm to (118.0, 124.5)

Commit message: update design
Parts:
- removed D1, D2: LED, LED_THT:LED_D5.0mm
- removed U5: W5500_Module, Custom Board:W5500_Module
- moved U6 126.2 mm to (56.5, 95.2)
- moved I6 8.68 mm to (55.9, 124.5)
- moved I5 1.27 mm to (114.3, 108.0)

Commit message: update design
Parts:
- added J1: Conn_01x02, Connector_JST:JST_XH_B2B-XH-A_1x02_P2.50mm_Vertical, F.Cu at (122.6, 89.5)
- moved U6 61.6 mm to (117.5, 104.1), turned to -90 degrees
- moved U3 25.0 mm to (60.3, 134.0)
- moved I3 23.7 mm to (122.0, 147.9), turned to 90 degrees
- moved I6 21.2 mm to (59.1, 103.5), turned to 90 degrees
- moved I4 20.9 mm to (90.2, 130.8)
- moved I5 19.3 mm to (97.2, 99.1), turned to 0 degrees
- moved U2 13.1 mm to (111.8, 133.4), turned to 90 degrees
- moved I2 9.91 mm to (111.8, 162.5), turned to 90 degrees
- moved I1 4.61 mm to (121.9, 162.6), turned to 90 degrees
- moved U4 3.94 mm to (121.9, 133.4), turned to 90 degrees
- moved U1 0.63 mm to (73.7, 156.8)
Connections:
- I1 pad 1: unconnected-(I1-GND-Pad1) -> GND
- I1 pad 2: unconnected-(I1-VCC-Pad2) -> +3V3
- I1 pad 3: unconnected-(I1-RX-Pad3) -> SO2_TX
- I1 pad 4: unconnected-(I1-TX-Pad4) -> SO2_RX
- I2 pad 1: unconnected-(I2-GND-Pad1) -> GND
- I2 pad 2: unconnected-(I2-VCC-Pad2) -> +3V3
- I2 pad 3: unconnected-(I2-RX-Pad3) -> H2S_TX
- I2 pad 4: unconnected-(I2-TX-Pad4) -> H2S_RX
- I3 pad 1: unconnected-(I3-GND-Pad1) -> GND
- I3 pad 2: unconnected-(I3-VCC-Pad2) -> +3V3
- I3 pad 3: unconnected-(I3-RX-Pad3) -> GPS_TX
- I3 pad 4: unconnected-(I3-TX-Pad4) -> GPS_RX
- I4 pad 1: unconnected-(I4-VCC-Pad1) -> +3V3
- I4 pad 2: unconnected-(I4-GND-Pad2) -> GND
- I4 pad 3: unconnected-(I4-SCL-Pad3) -> I2C_SCL
- I4 pad 4: unconnected-(I4-SDA-Pad4) -> I2C_SDA
- I5 pad 1: unconnected-(I5-VCC-Pad1) -> +3V3
- I5 pad 2: unconnected-(I5-GND-Pad2) -> GND
- I5 pad 3: unconnected-(I5-SCL-Pad3) -> I2C_SCL
- I5 pad 4: unconnected-(I5-SDA-Pad4) -> I2C_SDA
- I5 pad 5: unconnected-(I5-VIN--Pad5) -> Net-(I5-VIN-)
- I5 pad 6: unconnected-(I5-VIN+-Pad6) -> BMS_P+
- I6 pad 1: unconnected-(I6-GND-Pad1) -> GND
- I6 pad 2: unconnected-(I6-VCC-Pad2) -> +3V3
- I6 pad 3: unconnected-(I6-SDA-Pad3) -> I2C_SDA
- I6 pad 4: unconnected-(I6-SCL-Pad4) -> I2C_SCL
- I6 pad 5: unconnected-(I6-SQW-Pad5) -> RTC_INT_SQW
- U1 pad 12: unconnected-(U1-39-Pad12) -> SO2_RX
- U1 pad 13: unconnected-(U1-40-Pad13) -> SO2_TX
- U1 pad 14: unconnected-(U1-41-Pad14) -> GPS_RX
- U1 pad 15: unconnected-(U1-42-Pad15) -> GPS_TX
- U1 pad 16: unconnected-(U1-45-Pad16) -> H2S_RX
- U1 pad 17: unconnected-(U1-46-Pad17) -> H2S_TX
- U1 pad 2: unconnected-(U1-GND-Pad2) -> GND
- U1 pad 20: unconnected-(U1-3-Pad20) -> SPI_SCK
- U1 pad 22: unconnected-(U1-VDD_3V3-Pad22) -> +3V3
- U1 pad 23: unconnected-(U1-GND-Pad23) -> GND
- U1 pad 28: unconnected-(U1-20-Pad28) -> I2C_SCL
- U1 pad 30: unconnected-(U1-21-Pad30) -> I2C_SDA
- U1 pad 31: unconnected-(U1-19-Pad31) -> RTC_INT_SQW
- U1 pad 38: unconnected-(U1-6-Pad38) -> SD_CS
- U1 pad 39: unconnected-(U1-5-Pad39) -> SPI_MISO
- U1 pad 40: unconnected-(U1-4-Pad40) -> SPI_MOSI
- U1 pad 6: unconnected-(U1-33-Pad6) -> ADC_WIND_DIR
- U1 pad 7: unconnected-(U1-34-Pad7) -> ADC_ANEMOMETER
- U2 pad 1: unconnected-(U2-GND-Pad1) -> GND
- U2 pad 2: unconnected-(U2-VCC-Pad2) -> +3V3
- U2 pad 3: unconnected-(U2-ADC-Pad3) -> ADC_ANEMOMETER
- U3 pad 1: unconnected-(U3-GND-Pad1) -> GND
- U3 pad 2: unconnected-(U3-MISO-Pad2) -> SPI_MISO
- U3 pad 3: unconnected-(U3-CLK-Pad3) -> SPI_SCK
- U3 pad 4: unconnected-(U3-MOSI-Pad4) -> SPI_MOSI
- U3 pad 5: unconnected-(U3-CS-Pad5) -> SD_CS
- U3 pad 6: unconnected-(U3-3v3-Pad6) -> +3V3
- U4 pad 1: unconnected-(U4-GND-Pad1) -> GND
- U4 pad 2: unconnected-(U4-VCC-Pad2) -> +3V3
- U4 pad 3: unconnected-(U4-ADC-Pad3) -> ADC_WIND_DIR
- U6 pad 1: unconnected-(U6-IN+-Pad1) -> Net-(I5-VIN-)
- U6 pad 2: unconnected-(U6-IN--Pad2) -> BMS_P-
- U6 pad 3: Net-(D2-K) -> +3V3
- U6 pad 4: Net-(D2-A) -> GND
Routing:
- net +3V3: track 0.00 -> 189.9 mm
- net I2C_SDA: track 0.00 -> 98.4 mm, vias 0 -> 1
- net SO2_RX: track 0.00 -> 59.5 mm
- net I2C_SCL: track 0.00 -> 57.9 mm
- net GPS_RX: track 0.00 -> 47.4 mm
- net SO2_TX: track 0.00 -> 46.3 mm
- net GPS_TX: track 0.00 -> 43.7 mm
- net H2S_RX: track 0.00 -> 25.2 mm
- net H2S_TX: track 0.00 -> 21.3 mm
- net BMS_P+: track 0.00 -> 15.3 mm
- net BMS_P-: track 0.00 -> 9.94 mm
- net Net-(I5-VIN-): track 0.00 -> 7.62 mm

Commit message: update design
Parts:
- added BME280: BME280_Module_JST, Connector_JST:JST_XH_B4B-XH-A_1x04_P2.50mm_Vertical, F.Cu at (119.4, 81.3)
- added I2C: I2C_EXPANDER_JST, Connector_JST:JST_XH_B4B-XH-A_1x04_P2.50mm_Vertical, F.Cu at (119.4, 35.6)
- added I2C: I2C_EXPANDER_JST, Connector_JST:JST_XH_B4B-XH-A_1x04_P2.50mm_Vertical, F.Cu at (119.4, 50.9)
- added LIGHT: Light_Sensor_I2C_JST, Connector_JST:JST_XH_B4B-XH-A_1x04_P2.50mm_Vertical, F.Cu at (119.4, 66.1)
- moved J1 92.3 mm to (49.6, 33.0), turned to 0 degrees
- moved U6 74.0 mm to (56.5, 62.2), turned to 0 degrees
- moved I6 45.1 mm to (57.1, 148.6), turned to -90 degrees
- moved I4 43.2 mm to (91.4, 87.6)
- moved I5 41.2 mm to (58.4, 85.1), turned to 90 degrees
- moved U2 34.0 mm to (119.4, 100.3), turned to -90 degrees
- moved I2 32.5 mm to (119.3, 130.9), turned to -90 degrees
- moved U3 21.4 mm to (55.9, 113.0), turned to 90 degrees
- moved U4 18.1 mm to (119.3, 115.5), turned to -90 degrees
- moved U1 17.8 mm to (83.8, 142.2), turned to 0 degrees
- moved I3 3.30 mm to (119.3, 146.1), turned to -90 degrees
- moved I1 2.89 mm to (119.3, 161.4), turned to -90 degrees
Routing:
- net +3V3: track 189.9 -> 397.0 mm
- net I2C_SCL: track 57.9 -> 223.1 mm, vias 0 -> 1
- net I2C_SDA: track 98.4 -> 225.3 mm
- net ADC_ANEMOMETER: track 0.00 -> 65.2 mm
- net SPI_SCK: track 0.00 -> 55.8 mm
- net ADC_WIND_DIR: track 0.00 -> 52.4 mm
- net RTC_INT_SQW: track 0.00 -> 36.2 mm
- net SD_CS: track 0.00 -> 35.1 mm
- net SPI_MISO: track 0.00 -> 32.1 mm
- net BMS_P+: track 15.3 -> 43.2 mm
- net SPI_MOSI: track 0.00 -> 27.5 mm
- net SO2_RX: track 59.5 -> 45.4 mm
- net BMS_P-: track 9.94 -> 23.7 mm
- net GPS_RX: track 47.4 -> 38.2 mm
- net H2S_TX: track 21.3 -> 29.5 mm
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- added copper zone on B.Cu, net GND
- added copper zone on F.Cu, net GND
Other:
- outline, holes or cut-outs redrawn
- board text added: "3V3"
- board text added: "ADC"
- board text added: "GND"
- board text added: "RX"
- board text added: "SCL"
- board text added: "SDA"
- board text added: "SULFUR MONITORING"
- board text added: "TX"
- board text added: "VERSION: 0.0.1 DATE: 251205"
- board text added: "X"
- board text added: "pcb rapid prototype by STAS-RG"

Commit message: update drc
Parts:
- I1: footprint Custom Board:TB600B_SO2 -> Custom Board:TB600B_SO2_Module
- I2: footprint Custom Board:TB600C_H2S -> Custom Board:TB600C_H2S_Module
- I3: footprint Custom Board:uBlox_NEO-6M_JST -> Custom Board:uBlox_NEO-6M_Module_JST
- I4: footprint Custom Board:SSD1306_onBoard -> Custom Board:SSD1306_Module
- I5: footprint Custom Board:INA219 -> Custom Board:INA219_Module
- I6: footprint Custom Board:DS3231 -> Custom Board:DS3231_Module
- U1: footprint Custom Board:Heltec_WSL_V3_v1 -> Custom Board:Heltec_WSL_V3_Module
- U2: footprint Custom Board:STASRG_Anemometer -> Custom Board:STASRG_Anemometer_Module
- U3: footprint Custom Board:Micro_SDCARD_v2 -> Custom Board:Micro_SDCARD_v2_Module
- U4: footprint Custom Board:STASRG_Wind_Dir -> Custom Board:STASRG_Wind_Dir_Module
- renumbered BME280 to U5, LIGHT to U7, I2C to U8, I2C to U9
Routing:
- net Net-(I5-VIN-): track 0.00 -> 15.7 mm
- net BMS_P-: track 23.7 -> 26.2 mm
Changed lines of the file:
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@@
 	(net 48 "unconnected-(U2-NC-Pad4)")
 	(net 49 "unconnected-(U4-NC-Pad4)")
-	(footprint "Custom Board:uBlox_NEO-6M_JST"
+	(footprint "Custom Board:uBlox_NEO-6M_Module_JST"
 		(layer "F.Cu")
 		(at 119.29 146.05 -90)
@@
 		(descr "JST XH series connector, B4B-XH-A (http://www.jst-mfg.com/product/pdf/eng/eXH.pdf), generated with kicad-footprint-generator")
 		(tags "connector JST XH vertical")
-		(property "Reference" "I2C"
+		(property "Reference" "U9"
 			(at 3.75 5.08 90)
 			(layer "F.SilkS")
@@
 		)
 	)
-	(footprint "Custom Board:TB600C_H2S"
+	(footprint "Custom Board:TB600C_H2S_Module"
 		(layer "F.Cu")
 		(at 119.29 130.89 -90)
@@
 		(embedded_fonts no)
 	)
-	(footprint "Custom Board:SSD1306_onBoard"
+	(footprint "Custom Board:SSD1306_Module"
 		(layer "F.Cu")
 		(at 91.44 87.63)
@@
 		(embedded_fonts no)
 	)
-	(footprint "Custom Board:DS3231"
+	(footprint "Custom Board:DS3231_Module"
 		(layer "F.Cu")
 		(at 57.149999 148.59 -90)
@@
 		(pad "1" thru_hole rect
 			(at 17.78 5.079999 90)
-			(size 1.8 1.47)
+			(size 1.8 1.8)
 			(drill 1)
 			(layers "*.Cu" "*.Mask")
@@
 		(pad "7" thru_hole rect
 			(at -17.78 2.54 90)
-			(size 1.8 1.47)
+			(size 1.8 1.8)
 			(drill 1)
 			(layers "*.Cu" "*.Mask")
@@
 		)
 	)
-	(footprint "Custom Board:Heltec_WSL_V3_v1"
+	(footprint "Custom Board:Heltec_WSL_V3_Module"
 		(layer "F.Cu")
 		(at 83.82 142.24)
@@
 		(embedded_fonts no)
 	)
-	(footprint "Custom Board:Micro_SDCARD_v2"
+	(footprint "Custom Board:Micro_SDCARD_v2_Module"
 		(layer "F.Cu")
 		(at 55.88 113.03 90)
@@
 		(descr "JST XH series connector, B4B-XH-A (http://www.jst-mfg.com/product/pdf/eng/eXH.pdf), generated with kicad-footprint-generator")
 		(tags "connector JST XH vertical")
-		(property "Reference" "LIGHT"
+		(property "Reference" "U7"
 			(at 3.75 5.08 90)
 			(layer "F.SilkS")
@@
 		(descr "JST XH series connector, B4B-XH-A (http://www.jst-mfg.com/product/pdf/eng/eXH.pdf), generated with kicad-footprint-generator")
 		(tags "connector JST XH vertical")
-		(property "Reference" "I2C"
+		(property "Reference" "U8"
 			(at 3.75 5.08 90)
 			(layer "F.SilkS")
@@
 		)
 	)
-	(footprint "Custom Board:STASRG_Anemometer"
+	(footprint "Custom Board:STASRG_Anemometer_Module"
 		(layer "F.Cu")
 		(at 119.38 100.27 -90)
@@
 		(embedded_fonts no)
 	)
-	(footprint "Custom Board:STASRG_Wind_Dir"
+	(footprint "Custom Board:STASRG_Wind_Dir_Module"
 		(layer "F.Cu")
 		(at 119.29 115.51 -90)
@@
 		(embedded_fonts no)
 	)
-	(footprint "Custom Board:TB600B_SO2"
+	(footprint "Custom Board:TB600B_SO2_Module"
 		(layer "F.Cu")
 		(at 119.29 161.37 -90)
@@
 		(embedded_fonts no)
 	)
-	(footprint "Custom Board:INA219"
+	(footprint "Custom Board:INA219_Module"
 		(layer "F.Cu")
 		(at 58.42 85.09 90)
@@
 		(descr "JST XH series connector, B4B-XH-A (http://www.jst-mfg.com/product/pdf/eng/eXH.pdf), generated with kicad-footprint-generator")
 		(tags "connector JST XH vertical")
-		(property "Reference" "BME280"
-			(at 3.75 5.08 90)
+		(property "Reference" "U5"
+			(at 3.75 5.08 270)
 			(layer "F.SilkS")
 			(effects
@@
 	)
 	(segment
+		(start 54.61 71.12)
+		(end 54.61 76.2)
+		(width 1.016)
+		(layer "F.Cu")
+		(net 23)
+	)
+	(segment
+		(start 52.07 68.58)
+		(end 54.61 71.12)
+		(width 1.016)
+		(layer "F.Cu")
+		(net 23)
+	)
+	(segment
+		(start 47.625 68.58)
+		(end 52.07 68.58)
+		(width 1.016)
+		(layer "F.Cu")
+		(net 23)
+	)
+	(segment
+		(start 47.625 66.04)
+		(end 47.625 68.58)
+		(width 1.016)
+		(layer "F.Cu")
+		(net 23)
+	)
+	(segment
 		(start 52.07 33.02)
 		(end 52.07 76.2)
@@
 	)
 	(segment
+		(start 47.625 55.88)
+		(end 47.625 58.42)
+		(width 1.016)
+		(layer "B.Cu")
+		(net 41)
+	)
+	(segment
 		(start 47.625 41.275)
 		(end 49.57 39.33)
@@
 		(polygon
 			(pts
-				(xy 38.1 22.86) (xy 134.62 22.86) (xy 134.62 177.8) (xy 38.1 177.8)
+				(xy 35.56 20.32) (xy 137.16 20.32) (xy 137.16 182.88) (xy 35.56 182.88)
 			)
 		)
