File: pcb/design/05_sulfurmonitoring_design_v4_no_display/05_sulfurmonitoring_design_v4_no_display.kicad_pcb (KiCad board)
At the start: 2 copper layers, 90 x 150 mm, 17 parts, among them J1 Conn_01x02, U1 Heltec_WSL_V3, U10 BMS_2S_Module_1_v1, U2 Anemometer, U3 Micro_SDCARD_v2, U4 Wind_Direction, U5 BME280_Module_JST, U6 BUCK_MP1584_3V3, U7 Light_Sensor_I2C_JST, U8 I2C_EXPANDER_JST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

Commit message: Update 05_sulfurmonitoring_design_v4_no_display.kicad_pcb
Parts:
- renumbered J1 to BAT
Changed lines of the file:
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@@
 		(descr "JST XH series connector, B2B-XH-A (http://www.jst-mfg.com/product/pdf/eng/eXH.pdf), generated with kicad-footprint-generator")
 		(tags "connector JST XH vertical")
-		(property "Reference" "J1"
-			(at 1.25 -3.55 90)
+		(property "Reference" "BAT"
+			(at 1.25 -3.55 270)
 			(layer "F.SilkS")
 			(effects
